File: FSR_Floor_Sensor_POC/FSR_Floor_Sensor_POC.kicad_sch (KiCad schematic)
At the start: 45 parts, among them J1 DRDY Jumpers, J2 FSR Ribbon Connector, J3 CS Jumpers, J4 Stackable Header, U1 ADS1256, U2 ADG708, U3 ADG708, U4 REF6025xDGK

Commit message: initial layout
Parts:
- removed J4: Stackable Header, Connector_PinSocket_2.54mm:PinSocket_2x16_P2.54mm_Vertical, symbol Connector_Generic:Conn_02x16_Odd_Even
- added J5: MCU Interface, Connector_PinHeader_2.54mm:PinHeader_1x08_P2.54mm_Vertical, symbol Connector:Conn_01x08_Pin
- added J6: Stacking Pin Header 2x10, Connector_PinHeader_2.54mm:PinHeader_2x10_P2.54mm_Vertical, symbol Connector_Generic:Conn_02x10_Odd_Even
- J1, J3: footprint Connector_PinHeader_2.54mm:PinHeader_2x08_P2.54mm_Vertical -> Connector_PinHeader_1.27mm:PinHeader_2x08_P1.27mm_Vertical
- RESR1: value 5m -> 22m
Connections:
- net +3V3: now also J6.18 (Pin_18)
- net +5V: now also J6.17 (Pin_17)
- net ADC_CLK: now also J5.5 (Pin_5)
- net CS_0: now also J6.7 (Pin_7)
- net CS_1: now also J6.8 (Pin_8)
- net CS_2: now also J6.5 (Pin_5)
- net CS_3: now also J6.6 (Pin_6)
- net CS_4: now also J6.3 (Pin_3)
- net CS_5: now also J6.4 (Pin_4)
- net CS_6: now also J6.1 (Pin_1)
- net CS_7: now also J6.2 (Pin_2)
- net DRDY_N_0: now also J6.10 (Pin_10)
- net DRDY_N_1: now also J6.9 (Pin_9)
- net DRDY_N_2: now also J6.12 (Pin_12)
- net DRDY_N_3: now also J6.11 (Pin_11)
- net DRDY_N_4: now also J6.14 (Pin_14)
- net DRDY_N_5: now also J6.13 (Pin_13)
- net DRDY_N_6: now also J6.16 (Pin_16)
- net DRDY_N_7: now also J6.15 (Pin_15)
- net GND: now also J5.1 (Pin_1), J6.19 (Pin_19), J6.20 (Pin_20)
- net MUX_A0: now also J5.6 (Pin_6)
- net MUX_A1: now also J5.7 (Pin_7)
- net MUX_A2: now also J5.8 (Pin_8)
- net RSF_0: now also J2.15 (Pin_15); no longer J2.16 (Pin_16)
- net RSF_1: now also J2.13 (Pin_13); no longer J2.14 (Pin_14)
- net RSF_2: now also J2.11 (Pin_11); no longer J2.12 (Pin_12)
- net RSF_3: now also J2.9 (Pin_9); no longer J2.10 (Pin_10)
- net RSF_4: now also J2.7 (Pin_7); no longer J2.8 (Pin_8)
- net RSF_5: now also J2.5 (Pin_5); no longer J2.6 (Pin_6)
- net RSF_6: now also J2.3 (Pin_3); no longer J2.4 (Pin_4)
- net RSF_7: now also J2.1 (Pin_1); no longer J2.2 (Pin_2)
- net SPI_MISO: now also J5.2 (Pin_2)
- net SPI_MOSI: now also J5.3 (Pin_3)
- net SPI_SCLK: now also J5.4 (Pin_4)
- net VEXC_2V5: now also J2.10 (Pin_10), J2.12 (Pin_12), J2.14 (Pin_14), J2.16 (Pin_16), J2.2 (Pin_2), J2.4 (Pin_4), J2.6 (Pin_6), J2.8 (Pin_8); no longer J2.1 (Pin_1), J2.11 (Pin_11), J2.13 (Pin_13), J2.15 (Pin_15), J2.3 (Pin_3), J2.5 (Pin_5), J2.7 (Pin_7), J2.9 (Pin_9)
- no-connect marks 7 -> 2
