File: FSR Floor Sensor Circuit V2/FSR Floor Sensor Circuit V2.kicad_sch (KiCad schematic)
At the start: 2 parts, among them J1 Daughterboard Connector, J2 MCU Connector

Commit message: don't use a-b pin headers because pin numbering doesn't match footprint
Parts:
- J1: footprint (none) -> Connector_PinSocket_2.54mm:PinSocket_2x08_P2.54mm_Vertical
- J2: footprint (none) -> Connector_PinSocket_2.54mm:PinSocket_2x04_P2.54mm_Vertical
Changed lines of the file:
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@@
+	(wire
+		(pts
+			(xy 83.82 27.94) (xy 87.63 27.94)
+		)
+		(stroke
+			(width 0)
+			(type default)
+		)
+	)
 	(wire
 		(pts
@@
 		(pts
 			(xy 67.31 45.72) (xy 71.12 45.72)
-		)
-		(stroke
-			(width 0)
-			(type default)
-		)
-	)
-	(wire
-		(pts
-			(xy 87.63 27.94) (xy 83.82 27.94)
 		)
 		(stroke
@@
 			)
 		)
-		(property "Footprint" ""
+		(property "Footprint" "Connector_PinSocket_2.54mm:PinSocket_2x08_P2.54mm_Vertical"
 			(at 76.2 35.56 0)
 			(hide yes)
@@
 			)
 		)
-		(property "Footprint" ""
+		(property "Footprint" "Connector_PinSocket_2.54mm:PinSocket_2x04_P2.54mm_Vertical"
 			(at 77.47 72.39 0)
 			(hide yes)

Commit message: daughterboard PCB layout
Parts:
- added H1, H2, H3: MountingHole_Pad, MountingHole:MountingHole_3mm_Pad_TopBottom, symbol Mechanical:MountingHole_Pad
- added H4: MountingHole_Pad, MountingHole:MountingHole_3mm_Pad, symbol Mechanical:MountingHole_Pad
Connections:
- net FSR_Mux_0: now also J2.6 (Pin_6); no longer J2.2 (Pin_2)
- net FSR_Mux_2: now also J2.2 (Pin_2); no longer J2.6 (Pin_6)
- net GND: now also H1.1, H2.1, H3.1, H4.1
Other:
- note added: "Components are common to both the MCU and FSR boards"
- moved on the sheet: J1

Commit message: fix mounting hole and cleanup
Parts:
- H4: footprint MountingHole:MountingHole_3mm_Pad -> MountingHole:MountingHole_3mm_Pad_TopBottom
Changed lines of the file:
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@@
 			)
 		)
-		(property "Footprint" "MountingHole:MountingHole_3mm_Pad"
+		(property "Footprint" "MountingHole:MountingHole_3mm_Pad_TopBottom"
 			(at 76.2 111.76 0)
 			(hide yes)
