File: FSR Floor Sensor Circuit V2/FSR Floor Sensor Circuit V2.kicad_pcb (KiCad board)
At the start: 2 copper layers, 50 x 39 mm, 14 parts, among them J1 Daughterboard Connector, J2 MCU Connector, J3 Board Select Jumper, J4 FSR Ribbon Cable, J5 FSR Disable Jumper, U1 TMUX1308APWR

Commit message: add 10M board-sense resistor
Parts:
- added R3: 10M, Resistor_SMD:R_0805_2012Metric, F.Cu at (40.0, 132.4)
Routing:
- net /2V5_REF: track 61.2 -> 72.7 mm
- net /FSR Daughterboard/Selected_FSR: track 44.2 -> 46.4 mm
Changed lines of the file:
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@@
 		(embedded_fonts no)
 	)
+	(footprint "Resistor_SMD:R_0805_2012Metric"
+		(layer "F.Cu")
+		(at 40.05 132.4 -90)
+		(descr "Resistor SMD 0805 (2012 Metric), square (rectangular) end terminal, IPC-7351 nominal, (Body size source: IPC-SM-782 page 72, https://www.pcb-3d.com/wordpress/wp-content/uploads/ipc-sm-782a_amendment_1_and_2.pdf)")
+		(tags "resistor")
+		(property "Reference" "R3"
+			(at 2.75 -0.05 90)
+			(layer "F.SilkS")
+			(effects
+				(font
+					(size 1 1)
+					(thickness 0.15)
+				)
+			)
+		)
+		(property "Value" "10M"
+			(at 0 1.65 90)
+			(layer "F.Fab")
+			(effects
+				(font
+					(size 1 1)
+					(thickness 0.15)
+				)
+			)
+		)
+		(property "Datasheet" ""
+			(at 0 0 90)
+			(layer "F.Fab")
+			(hide yes)
+			(effects
+				(font
+					(size 1.27 1.27)
+				)
+			)
+		)
+		(property "Description" "Resistor"
+			(at 0 0 90)
+			(layer "F.Fab")
+			(hide yes)
+			(effects
+				(font
+					(size 1.27 1.27)
+				)
+			)
+		)
+		(property ki_fp_filters "R_*")
+		(sheetname "/FSR Daughterboard/")
+		(sheetfile "fsr_daughterboard.kicad_sch")
+		(units
+			(unit
+				(name "A")
+				(pins "1" "2")
+			)
+		)
+		(attr smd)
+		(duplicate_pad_numbers_are_jumpers no)
+		(fp_line
+			(start -0.227064 0.735)
+			(end 0.227064 0.735)
+			(stroke
+				(width 0.12)
+				(type solid)
+			)
+			(layer "F.SilkS")
+		)
+		(fp_line
+			(start -0.227064 -0.735)
+			(end 0.227064 -0.735)
+			(stroke
+				(width 0.12)
+				(type solid)
+			)
+			(layer "F.SilkS")
+		)
+		(fp_rect
+			(start -1.68 -0.95)
+			(end 1.68 0.95)
+			(stroke
+				(width 0.05)
+				(type solid)
+			)
+			(fill no)
+			(layer "F.CrtYd")
+		)
+		(fp_rect
+			(start -1 -0.625)
+			(end 1 0.625)
+			(stroke
+				(width 0.1)
+				(type solid)
+			)
+			(fill no)
+			(layer "F.Fab")
+		)
+		(fp_text user "${REFERENCE}"
+			(at 0 0 90)
+			(layer "F.Fab")
+			(effects
+				(font
+					(size 0.5 0.5)
+					(thickness 0.08)
+				)
+			)
+		)
+		(pad "1" smd roundrect
+			(at -0.9125 0 270)
+			(size 1.025 1.4)
+			(layers "F.Cu" "F.Mask" "F.Paste")
+			(roundrect_rratio 0.243902)
+			(net "/FSR Daughterboard/Selected_FSR")
+			(pintype "passive")
+		)
+		(pad "2" smd roundrect
+			(at 0.9125 0 270)
+			(size 1.025 1.4)
+			(layers "F.Cu" "F.Mask" "F.Paste")
+			(roundrect_rratio 0.243902)
+			(net "/2V5_REF")
+			(pintype "passive")
+		)
+		(embedded_fonts no)
+		(model "${KICAD10_3DMODEL_DIR}/Resistor_SMD.3dshapes/R_0805_2012Metric.step"
+			(offset
+				(xyz 0 0 0)
+			)
+			(scale
+				(xyz 1 1 1)
+			)
+			(rotate
+				(xyz 0 0 0)
+			)
+		)
+	)
 	(footprint "Capacitor_SMD:C_0805_2012Metric"
 		(layer "F.Cu")
@@
 	)
 	(segment
-		(start 37.07 129.195536)
+		(start 40.05 129.195536)
 		(end 41.795536 129.195536)
 		(width 0.2)
@@
 	)
 	(segment
+		(start 37.07 129.195536)
+		(end 40.05 129.195536)
+		(width 0.2)
+		(layer "F.Cu")
+		(net "/FSR Daughterboard/Selected_FSR")
+	)
+	(segment
 		(start 57.265 125.565)
 		(end 56.15 125.565)
@@
 	)
 	(segment
+		(start 40.05 131.4875)
+		(end 40.05 129.195536)
+		(width 0.2)
+		(layer "F.Cu")
+		(net "/FSR Daughterboard/Selected_FSR")
+	)
+	(segment
 		(start 37.07 119.035536)
 		(end 37.07 138.085536)
@@
 	)
 	(segment
+		(start 40.05 138.02)
+		(end 40.05 133.3125)
+		(width 0.5)
+		(layer "F.Cu")
+		(net "/2V5_REF")
+	)
+	(segment
 		(start 64.72 142.82)
 		(end 64.75 142.85)
@@
 		(width 0.5)
 		(layer "F.Cu")
+		(net "/2V5_REF")
+	)
+	(segment
+		(start 44.85 142.82)
+		(end 40.05 138.02)
+		(width 0.5)
+		(layer "F.Cu")
