File: FSR Floor Sensor Circuit V2/fsr_daughterboard.kicad_sch (KiCad schematic)
At the start: 6 parts, among them J3 Board Select Jumper, J4 FSR Ribbon Cable, J5 FSR Disable Jumper, U1 TMUX1308APWR

Commit message: don't use a-b pin headers because pin numbering doesn't match footprint
Parts:
- C1: footprint (none) -> Capacitor_SMD:C_0805_2012Metric
- J3: footprint (none) -> Connector_PinHeader_1.27mm:PinHeader_2x16_P1.27mm_Vertical; symbol Connector_Generic:Conn_02x16_Row_Letter_Last -> Connector_Generic:Conn_02x16_Odd_Even
- J4: footprint (none) -> Connector_IDC:IDC-Header_2x08_P2.54mm_Vertical; symbol Connector_Generic:Conn_02x08_Row_Letter_Last -> Connector_Generic:Conn_02x08_Odd_Even
- J5: footprint (none) -> Connector_PinHeader_1.27mm:PinHeader_2x08_P1.27mm_Vertical; symbol Connector_Generic:Conn_02x08_Row_Letter_Last -> Connector_Generic:Conn_02x08_Odd_Even
- R_DIS1: footprint (none) -> Resistor_SMD:R_0805_2012Metric
Connections:
- net 2V5_REF: now also J4.1 (Pin_1), J4.11 (Pin_11), J4.13 (Pin_13), J4.15 (Pin_15), J4.3 (Pin_3), J4.5 (Pin_5), J4.7 (Pin_7), J4.9 (Pin_9); no longer J4.1a (Pin_1a), J4.2a (Pin_2a), J4.3a (Pin_3a), J4.4a (Pin_4a), J4.5a (Pin_5a), J4.6a (Pin_6a), J4.7a (Pin_7a), J4.8a (Pin_8a)
- net Daughter_1: now also J3.1 (Pin_1); no longer J3.1a (Pin_1a)
- net Daughter_10: now also J3.19 (Pin_19); no longer J3.10a (Pin_10a)
- net Daughter_11: now also J3.21 (Pin_21); no longer J3.11a (Pin_11a)
- net Daughter_12: now also J3.23 (Pin_23); no longer J3.12a (Pin_12a)
- net Daughter_13: now also J3.25 (Pin_25); no longer J3.13a (Pin_13a)
- net Daughter_14: now also J3.27 (Pin_27); no longer J3.14a (Pin_14a)
- net Daughter_15: now also J3.29 (Pin_29); no longer J3.15a (Pin_15a)
- net Daughter_16: now also J3.31 (Pin_31); no longer J3.16a (Pin_16a)
- net Daughter_2: now also J3.3 (Pin_3); no longer J3.2a (Pin_2a)
- net Daughter_3: now also J3.5 (Pin_5); no longer J3.3a (Pin_3a)
- net Daughter_4: now also J3.7 (Pin_7); no longer J3.4a (Pin_4a)
- net Daughter_5: now also J3.9 (Pin_9); no longer J3.5a (Pin_5a)
- net Daughter_6: now also J3.11 (Pin_11); no longer J3.6a (Pin_6a)
- net Daughter_7: now also J3.13 (Pin_13); no longer J3.7a (Pin_7a)
- net Daughter_8: now also J3.15 (Pin_15); no longer J3.8a (Pin_8a)
- net Daughter_9: now also J3.17 (Pin_17); no longer J3.9a (Pin_9a)
- net FSR_1: now also J4.2 (Pin_2), J5.1 (Pin_1); no longer J4.1b (Pin_1b), J5.1a (Pin_1a)
- net FSR_2: now also J4.4 (Pin_4), J5.3 (Pin_3); no longer J4.2b (Pin_2b), J5.2a (Pin_2a)
- net FSR_3: now also J4.6 (Pin_6), J5.5 (Pin_5); no longer J4.3b (Pin_3b), J5.3a (Pin_3a)
- net FSR_4: now also J4.8 (Pin_8), J5.7 (Pin_7); no longer J4.4b (Pin_4b), J5.4a (Pin_4a)
- net FSR_5: now also J4.10 (Pin_10), J5.9 (Pin_9); no longer J4.5b (Pin_5b), J5.5a (Pin_5a)
- net FSR_6: now also J4.12 (Pin_12), J5.11 (Pin_11); no longer J4.6b (Pin_6b), J5.6a (Pin_6a)
- net FSR_7: now also J4.14 (Pin_14), J5.13 (Pin_13); no longer J4.7b (Pin_7b), J5.7a (Pin_7a)
- net FSR_8: now also J4.16 (Pin_16), J5.15 (Pin_15); no longer J4.8b (Pin_8b), J5.8a (Pin_8a)
- net FSR_DIS: now also J5.10 (Pin_10), J5.12 (Pin_12), J5.14 (Pin_14), J5.16 (Pin_16), J5.2 (Pin_2), J5.4 (Pin_4), J5.6 (Pin_6), J5.8 (Pin_8); no longer J5.1b (Pin_1b), J5.2b (Pin_2b), J5.3b (Pin_3b), J5.4b (Pin_4b), J5.5b (Pin_5b), J5.6b (Pin_6b), J5.7b (Pin_7b), J5.8b (Pin_8b)
- net Selected_FSR: now also J3.10 (Pin_10), J3.12 (Pin_12), J3.14 (Pin_14), J3.16 (Pin_16), J3.18 (Pin_18), J3.2 (Pin_2), J3.20 (Pin_20), J3.22 (Pin_22), J3.24 (Pin_24), J3.26 (Pin_26), J3.28 (Pin_28), J3.30 (Pin_30), J3.32 (Pin_32), J3.4 (Pin_4), J3.6 (Pin_6), J3.8 (Pin_8); no longer J3.10b (Pin_10b), J3.11b (Pin_11b), J3.12b (Pin_12b), J3.13b (Pin_13b), J3.14b (Pin_14b), J3.15b (Pin_15b), J3.16b (Pin_16b), J3.1b (Pin_1b), J3.2b (Pin_2b), J3.3b (Pin_3b), J3.4b (Pin_4b), J3.5b (Pin_5b), J3.6b (Pin_6b), J3.7b (Pin_7b), J3.8b (Pin_8b), J3.9b (Pin_9b)

Commit message: daughterboard PCB layout
Parts:
- added FID1, FID2: Fiducial, Fiducial:Fiducial_1mm_Mask2mm, symbol Mechanical:Fiducial
- J5: footprint Connector_PinHeader_1.27mm:PinHeader_2x08_P1.27mm_Vertical -> Connector_PinHeader_2.54mm:PinHeader_2x08_P2.54mm_Vertical
Connections:
- net FSR_1: now also J5.2 (Pin_2); no longer J5.1 (Pin_1)
- net FSR_2: now also J5.4 (Pin_4); no longer J5.3 (Pin_3)
- net FSR_3: now also J5.6 (Pin_6); no longer J5.5 (Pin_5)
- net FSR_4: now also J5.8 (Pin_8); no longer J5.7 (Pin_7)
- net FSR_5: now also J5.10 (Pin_10); no longer J5.9 (Pin_9)
- net FSR_6: now also J5.12 (Pin_12); no longer J5.11 (Pin_11)
- net FSR_7: now also J5.14 (Pin_14); no longer J5.13 (Pin_13)
- net FSR_8: now also J5.16 (Pin_16); no longer J5.15 (Pin_15)
- net FSR_DIS: now also J5.1 (Pin_1), J5.11 (Pin_11), J5.13 (Pin_13), J5.15 (Pin_15), J5.3 (Pin_3), J5.5 (Pin_5), J5.7 (Pin_7), J5.9 (Pin_9); no longer J5.10 (Pin_10), J5.12 (Pin_12), J5.14 (Pin_14), J5.16 (Pin_16), J5.2 (Pin_2), J5.4 (Pin_4), J5.6 (Pin_6), J5.8 (Pin_8)
Changed lines of the file:
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@@
+	(wire
+		(pts
+			(xy 110.49 82.55) (xy 107.95 82.55)
+		)
+		(stroke
+			(width 0)
+			(type default)
+		)
+	)
+	(wire
+		(pts
+			(xy 97.79 53.34) (xy 97.79 55.88)
+		)
+		(stroke
+			(width 0)
+			(type default)
+		)
+	)
+	(wire
+		(pts
+			(xy 66.04 48.26) (xy 82.55 48.26)
+		)
+		(stroke
+			(width 0)
+			(type default)
+		)
+	)
+	(wire
+		(pts
+			(xy 132.08 30.48) (xy 147.32 30.48)
+		)
+		(stroke
+			(width 0)
+			(type default)
+		)
+	)
+	(bus
+		(pts
+			(xy 63.5 25.4) (xy 63.5 30.48)
+		)
+		(stroke
+			(width 0)
+			(type default)
+		)
+	)
+	(wire
+		(pts
+			(xy 173.99 43.18) (xy 170.18 43.18)
+		)
+		(stroke
+			(width 0)
+			(type default)
+		)
+	)
+	(wire
+		(pts
+			(xy 97.79 33.02) (xy 95.25 33.02)
+		)
+		(stroke
+			(width 0)
+			(type default)
+		)
+	)
+	(bus
+		(pts
+			(xy 63.5 48.26) (xy 63.5 50.8)
+		)
+		(stroke
+			(width 0)
+			(type default)
+		)
+	)
+	(wire
+		(pts
+			(xy 110.49 85.09) (xy 107.95 85.09)
+		)
+		(stroke
+			(width 0)
+			(type default)
+		)
+	)
+	(wire
+		(pts
+			(xy 170.18 34.29) (xy 170.18 30.48)
+		)
+		(stroke
+			(width 0)
+			(type default)
+		)
+	)
 	(wire
 		(pts
 			(xy 170.18 43.18) (xy 170.18 73.66)
-		)
-		(stroke
-			(width 0)
-			(type default)
-		)
-	)
-	(wire
-		(pts
-			(xy 110.49 82.55) (xy 107.95 82.55)
-		)
-		(stroke
-			(width 0)
-			(type default)
-		)
-	)
-	(wire
-		(pts
-			(xy 97.79 53.34) (xy 97.79 55.88)
-		)
-		(stroke
-			(width 0)
-			(type default)
-		)
-	)
-	(wire
-		(pts
-			(xy 66.04 48.26) (xy 82.55 48.26)
-		)
-		(stroke
-			(width 0)
-			(type default)
-		)
-	)
-	(wire
-		(pts
-			(xy 132.08 30.48) (xy 147.32 30.48)
-		)
-		(stroke
-			(width 0)
-			(type default)
-		)
-	)
-	(bus
-		(pts
-			(xy 63.5 25.4) (xy 63.5 30.48)
-		)
-		(stroke
-			(width 0)
-			(type default)
-		)
-	)
-	(wire
-		(pts
-			(xy 173.99 43.18) (xy 170.18 43.18)
-		)
-		(stroke
-			(width 0)
-			(type default)
-		)
-	)
-	(wire
-		(pts
-			(xy 97.79 33.02) (xy 95.25 33.02)
-		)
-		(stroke
-			(width 0)
-			(type default)
-		)
-	)
-	(bus
-		(pts
-			(xy 63.5 48.26) (xy 63.5 50.8)
-		)
-		(stroke
-			(width 0)
-			(type default)
-		)
-	)
-	(wire
-		(pts
-			(xy 110.49 85.09) (xy 107.95 85.09)
-		)
-		(stroke
-			(width 0)
-			(type default)
-		)
-	)
-	(wire
-		(pts
-			(xy 170.18 34.29) (xy 170.18 30.48)
 		)
 		(stroke
@@
 	(symbol
 		(lib_id "Connector_Generic:Conn_02x08_Odd_Even")
-		(at 100.33 87.63 0)
+		(at 102.87 87.63 0)
+		(mirror y)
 		(unit 1)
 		(body_style 1)
@@
 		(in_pos_files yes)
 		(dnp no)
-		(fields_autoplaced yes)
 		(property "Reference" "J5"
-			(at 101.6 73.66 0)
+			(at 101.6 88.9 0)
 			(show_name no)
 			(do_not_autoplace no)
@@
 			)
 		)
-		(property "Footprint" "Connector_PinHeader_1.27mm:PinHeader_2x08_P1.27mm_Vertical"
-			(at 100.33 87.63 0)
+		(property "Footprint" "Connector_PinHeader_2.54mm:PinHeader_2x08_P2.54mm_Vertical"
+			(at 102.87 87.63 0)
 			(hide yes)
 			(show_name no)
@@
 		)
 		(property "Datasheet" ""
-			(at 100.33 87.63 0)
+			(at 102.87 87.63 0)
 			(hide yes)
 			(show_name no)
@@
 		)
 		(property "Description" "Generic connector, double row, 02x08, odd/even pin numbering scheme (row 1 odd numbers, row 2 even numbers), script generated (kicad-library-utils/schlib/autogen/connector/)"
-			(at 100.33 87.63 0)
+			(at 102.87 87.63 0)
 			(hide yes)
 			(show_name no)
@@
 		(in_pos_files yes)
 		(dnp no)
-		(fields_autoplaced yes)
 		(property "Reference" "J4"
-			(at 74.93 73.66 0)
+			(at 74.93 88.9 0)
 			(show_name no)
 			(do_not_autoplace no)
@@
 				(path "/f755b232-d3a3-432e-82d0-c24f93d5f8c8/4081d15f-10c6-4ec3-98a3-c3d13b71b01e"
 					(reference "R_DIS1")
+					(unit 1)
+				)
+			)
+		)
+	)
+	(symbol
+		(lib_id "Mechanical:Fiducial")
+		(at 119.38 63.5 0)
+		(unit 1)
+		(body_style 1)
+		(exclude_from_sim no)
+		(in_bom no)
+		(on_board yes)
+		(in_pos_files yes)
+		(dnp no)
+		(fields_autoplaced yes)
+		(property "Reference" "FID2"
+			(at 121.92 62.2299 0)
+			(show_name no)
+			(do_not_autoplace no)
+			(effects
+				(font
+					(size 1.27 1.27)
+				)
+				(justify left)
+			)
+		)
+		(property "Value" "Fiducial"
+			(at 121.92 64.7699 0)
+			(show_name no)
+			(do_not_autoplace no)
+			(effects
+				(font
+					(size 1.27 1.27)
+				)
+				(justify left)
+			)
+		)
+		(property "Footprint" "Fiducial:Fiducial_1mm_Mask2mm"
+			(at 119.38 63.5 0)
+			(hide yes)
+			(show_name no)
+			(do_not_autoplace no)
+			(effects
+				(font
+					(size 1.27 1.27)
+				)
+			)
+		)
+		(property "Datasheet" ""
+			(at 119.38 63.5 0)
+			(hide yes)
+			(show_name no)
+			(do_not_autoplace no)
+			(effects
+				(font
+					(size 1.27 1.27)
+				)
+			)
+		)
+		(property "Description" "Fiducial Marker"
+			(at 119.38 63.5 0)
+			(hide yes)
+			(show_name no)
+			(do_not_autoplace no)
+			(effects
+				(font
+					(size 1.27 1.27)
+				)
+			)
+		)
+		(instances
+			(project "FSR Floor Sensor Circuit V2"
+				(path "/f755b232-d3a3-432e-82d0-c24f93d5f8c8/4081d15f-10c6-4ec3-98a3-c3d13b71b01e"
+					(reference "FID2")
 					(unit 1)
 				)
@@
 					(unit 1)
 				)
+			)
+		)
+	)
+	(symbol
+		(lib_id "Mechanical:Fiducial")
+		(at 109.22 53.34 0)
+		(unit 1)
+		(body_style 1)
+		(exclude_from_sim no)
+		(in_bom no)
+		(on_board yes)
+		(in_pos_files yes)
+		(dnp no)
+		(fields_autoplaced yes)
+		(property "Reference" "FID1"
+			(at 111.76 52.0699 0)
+			(show_name no)
+			(do_not_autoplace no)
+			(effects
+				(font
+					(size 1.27 1.27)
+				)
+				(justify left)
+			)
+		)
+		(property "Value" "Fiducial"
+			(at 111.76 54.6099 0)
+			(show_name no)
+			(do_not_autoplace no)
+			(effects
+				(font
+					(size 1.27 1.27)
+				)
+				(justify left)
+			)
+		)
+		(property "Footprint" "Fiducial:Fiducial_1mm_Mask2mm"
+			(at 109.22 53.34 0)
+			(hide yes)
+			(show_name no)
+			(do_not_autoplace no)
+			(effects
+				(font
+					(size 1.27 1.27)
+				)
+			)
+		)
+		(property "Datasheet" ""
+			(at 109.22 53.34 0)
+			(hide yes)
+			(show_name no)
+			(do_not_autoplace no)
+			(effects
+				(font
+					(size 1.27 1.27)
+				)
+			)
+		)
+		(property "Description" "Fiducial Marker"
+			(at 109.22 53.34 0)
+			(hide yes)
+			(show_name no)
+			(do_not_autoplace no)
+			(effects
+				(font
+					(size 1.27 1.27)
+				)
+			)
+		)
+		(instances
+			(project "FSR Floor Sensor Circuit V2"
+				(path "/f755b232-d3a3-432e-82d0-c24f93d5f8c8/4081d15f-10c6-4ec3-98a3-c3d13b71b01e"
+					(reference "FID1")
+					(unit 1)
+				)

Commit message: add 10M board-sense resistor
Parts:
- added R3: 10M, Resistor_SMD:R_0805_2012Metric, symbol Device:R
Connections:
- net 2V5_REF: now also R3.2
- net Selected_FSR: now also R3.1
Other:
- note added: "board-detection resistor"
- moved on the sheet: FID1, FID2
Changed lines of the file:
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@@
 	(generator_version "10.0")
 	(paper "A4")
+	(text "board-detection resistor"
+		(exclude_from_sim no)
+		(at 121.92 58.42 90)
+		(effects
+			(font
+				(size 1.27 1.27)
+			)
+		)
+	)
 	(junction
 		(at 97.79 60.96)
@@
 	(junction
 		(at 66.04 85.09)
+		(diameter 0)
+		(color 0 0 0 0)
+	)
+	(junction
+		(at 125.73 43.18)
 		(diameter 0)
 		(color 0 0 0 0)
@@
 	(wire
 		(pts
+			(xy 125.73 45.72) (xy 125.73 43.18)
+		)
+		(stroke
+			(width 0)
+			(type default)
+		)
+	)
+	(wire
+		(pts
 			(xy 97.79 60.96) (xy 95.25 60.96)
 		)
@@
 	(wire
 		(pts
+			(xy 125.73 55.88) (xy 125.73 53.34)
+		)
+		(stroke
+			(width 0)
+			(type default)
+		)
+	)
+	(wire
+		(pts
 			(xy 81.28 97.79) (xy 95.25 97.79)
 		)
@@
 	(wire
 		(pts
+			(xy 125.73 43.18) (xy 147.32 43.18)
+		)
+		(stroke
+			(width 0)
+			(type default)
+		)
+	)
+	(wire
+		(pts
 			(xy 110.49 82.55) (xy 107.95 82.55)
 		)
@@
 	(wire
 		(pts
-			(xy 97.79 43.18) (xy 147.32 43.18)
+			(xy 97.79 43.18) (xy 125.73 43.18)
 		)
 		(stroke
@@
 		(shape input)
 		(at 124.46 25.4 180)
+		(effects
+			(font
+				(size 1.27 1.27)
+			)
+			(justify right)
+		)
+	)
+	(hierarchical_label "2V5_REF"
+		(shape input)
+		(at 125.73 55.88 270)
 		(effects
 			(font
@@
 	(symbol
 		(lib_id "Mechanical:Fiducial")
-		(at 119.38 63.5 0)
+		(at 137.16 93.98 0)
 		(unit 1)
 		(body_style 1)
@@
 		(fields_autoplaced yes)
 		(property "Reference" "FID2"
-			(at 121.92 62.2299 0)
+			(at 139.7 92.7099 0)
 			(show_name no)
 			(do_not_autoplace no)
@@
 		)
 		(property "Value" "Fiducial"
-			(at 121.92 64.7699 0)
+			(at 139.7 95.2499 0)
 			(show_name no)
 			(do_not_autoplace no)
@@
 		)
 		(property "Footprint" "Fiducial:Fiducial_1mm_Mask2mm"
-			(at 119.38 63.5 0)
+			(at 137.16 93.98 0)
 			(hide yes)
 			(show_name no)
@@
 		)
 		(property "Datasheet" ""
-			(at 119.38 63.5 0)
+			(at 137.16 93.98 0)
 			(hide yes)
 			(show_name no)
@@
 		)
 		(property "Description" "Fiducial Marker"
-			(at 119.38 63.5 0)
+			(at 137.16 93.98 0)
 			(hide yes)
 			(show_name no)
@@
 	)
 	(symbol
+		(lib_id "Device:R")
+		(at 125.73 49.53 0)
+		(unit 1)
+		(body_style 1)
+		(exclude_from_sim no)
+		(in_bom yes)
+		(on_board yes)
+		(in_pos_files yes)
+		(dnp no)
+		(fields_autoplaced yes)
+		(property "Reference" "R3"
+			(at 128.27 48.2599 0)
+			(show_name no)
+			(do_not_autoplace no)
+			(effects
+				(font
+					(size 1.27 1.27)
+				)
+				(justify left)
+			)
+		)
+		(property "Value" "10M"
+			(at 128.27 50.7999 0)
+			(show_name no)
+			(do_not_autoplace no)
+			(effects
+				(font
+					(size 1.27 1.27)
+				)
+				(justify left)
+			)
+		)
+		(property "Footprint" "Resistor_SMD:R_0805_2012Metric"
+			(at 123.952 49.53 90)
+			(hide yes)
+			(show_name no)
+			(do_not_autoplace no)
+			(effects
+				(font
+					(size 1.27 1.27)
+				)
+			)
+		)
+		(property "Datasheet" ""
+			(at 125.73 49.53 0)
+			(hide yes)
+			(show_name no)
+			(do_not_autoplace no)
+			(effects
+				(font
+					(size 1.27 1.27)
+				)
+			)
+		)
+		(property "Description" "Resistor"
+			(at 125.73 49.53 0)
+			(hide yes)
+			(show_name no)
+			(do_not_autoplace no)
+			(effects
+				(font
+					(size 1.27 1.27)
+				)
+			)
+		)
+		(pin "2"
+		)
+		(pin "1"
+		)
+		(instances
+			(project "FSR Floor Sensor Circuit V2"
+				(path "/f755b232-d3a3-432e-82d0-c24f93d5f8c8/4081d15f-10c6-4ec3-98a3-c3d13b71b01e"
+					(reference "R3")
+					(unit 1)
+				)
+			)
+		)
+	)
+	(symbol
 		(lib_id "Mechanical:Fiducial")
-		(at 109.22 53.34 0)
+		(at 127 83.82 0)
 		(unit 1)
 		(body_style 1)
@@
 		(fields_autoplaced yes)
 		(property "Reference" "FID1"
-			(at 111.76 52.0699 0)
+			(at 129.54 82.5499 0)
 			(show_name no)
 			(do_not_autoplace no)
@@
 		)
 		(property "Value" "Fiducial"
-			(at 111.76 54.6099 0)
+			(at 129.54 85.0899 0)
 			(show_name no)
 			(do_not_autoplace no)
@@
 		)
 		(property "Footprint" "Fiducial:Fiducial_1mm_Mask2mm"
-			(at 109.22 53.34 0)
+			(at 127 83.82 0)
 			(hide yes)
 			(show_name no)
@@
 		)
 		(property "Datasheet" ""
-			(at 109.22 53.34 0)
+			(at 127 83.82 0)
 			(hide yes)
 			(show_name no)
@@
 		)
 		(property "Description" "Fiducial Marker"
-			(at 109.22 53.34 0)
-			(hide yes)
-			(show_name no)
+			(at 127 83.82 0)
+			(hide yes)
+			(show_name no)
